File: hardware/_saved_hardware.sch (KiCad schematic (older format))
At the start: 16 parts, among them J1 Raspberry_Pi_2_3, J2 SSD1608_SPI, J3 0906-1, J4 0906-1, J5 Batt, J6 USB_A, U1 MCP73871, U2 L7805

Commit message: update pcb
Parts:
- J1: footprint Connector_PinHeader_2.54mm:PinHeader_2x20_P2.54mm_Vertical -> Connector_PinSocket_2.54mm:PinSocket_2x20_P2.54mm_Vertical
- R1, R2, R3, R4, R5, R6: footprint Resistor_SMD:R_1020_2550Metric -> Resistor_SMD:R_0805_2012Metric
- SW1: renamed from SW?; footprint (none) -> Button_Switch_THT:SW_PUSH_6mm
Changed lines of the file:
@@
 F 0 "J1" H 3200 4428 50  0000 C CNN
 F 1 "Raspberry_Pi_2_3" H 3200 4337 50  0000 C CNN
-F 2 "Connector_PinHeader_2.54mm:PinHeader_2x20_P2.54mm_Vertical" H 3200 2950 50  0001 C CNN
+F 2 "Connector_PinSocket_2.54mm:PinSocket_2x20_P2.54mm_Vertical" H 3200 2950 50  0001 C CNN
 F 3 "https://www.raspberrypi.org/documentation/hardware/raspberrypi/schematics/rpi_SCH_3bplus_1p0_reduced.pdf" H 3200 2950 50  0001 C CNN
 	1    3200 2950
@@
 F 0 "R3" H 7870 4546 50  0000 L CNN
 F 1 "100K" H 7870 4455 50  0000 L CNN
-F 2 "Resistor_SMD:R_1020_2550Metric" V 7730 4500 50  0001 C CNN
+F 2 "Resistor_SMD:R_0805_2012Metric" V 7730 4500 50  0001 C CNN
 F 3 "~" H 7800 4500 50  0001 C CNN
 	1    7800 4500
@@
 F 0 "R2" H 7870 4146 50  0000 L CNN
 F 1 "270k" H 7870 4055 50  0000 L CNN
-F 2 "Resistor_SMD:R_1020_2550Metric" V 7730 4100 50  0001 C CNN
+F 2 "Resistor_SMD:R_0805_2012Metric" V 7730 4100 50  0001 C CNN
 F 3 "~" H 7800 4100 50  0001 C CNN
 	1    7800 4100
@@
 F 0 "R1" H 7500 5200 50  0000 L CNN
 F 1 "2K" H 7500 5100 50  0000 L CNN
-F 2 "Resistor_SMD:R_1020_2550Metric" V 7580 5150 50  0001 C CNN
+F 2 "Resistor_SMD:R_0805_2012Metric" V 7580 5150 50  0001 C CNN
 F 3 "~" H 7650 5150 50  0001 C CNN
 	1    7650 5150
@@
 F 0 "R5" H 7750 5200 50  0000 L CNN
 F 1 "100K" H 7750 5100 50  0000 L CNN
-F 2 "Resistor_SMD:R_1020_2550Metric" V 7830 5150 50  0001 C CNN
+F 2 "Resistor_SMD:R_0805_2012Metric" V 7830 5150 50  0001 C CNN
 F 3 "~" H 7900 5150 50  0001 C CNN
 	1    7900 5150
@@
 F 0 "R6" H 8120 5996 50  0000 L CNN
 F 1 "150K" H 8120 5905 50  0000 L CNN
-F 2 "Resistor_SMD:R_1020_2550Metric" V 7980 5950 50  0001 C CNN
+F 2 "Resistor_SMD:R_0805_2012Metric" V 7980 5950 50  0001 C CNN
 F 3 "~" H 8050 5950 50  0001 C CNN
 	1    8050 5950
@@
 F 0 "R4" H 7870 5996 50  0000 L CNN
 F 1 "10K" H 7870 5905 50  0000 L CNN
-F 2 "Resistor_SMD:R_1020_2550Metric" V 7730 5950 50  0001 C CNN
+F 2 "Resistor_SMD:R_0805_2012Metric" V 7730 5950 50  0001 C CNN
 F 3 "~" H 7800 5950 50  0001 C CNN
 	1    7800 5950
@@
 	1700 3300 1700 3100
 $Comp
-L Switch:SW_MEC_5G SW?
+L Switch:SW_MEC_5G SW1
 U 1 1 5BD68F4E
 P 1450 3300
-F 0 "SW?" H 1450 3585 50  0000 C CNN
+F 0 "SW1" H 1450 3585 50  0000 C CNN
 F 1 "SW_MEC_5G" H 1450 3494 50  0000 C CNN
-F 2 "" H 1450 3500 50  0001 C CNN
+F 2 "Button_Switch_THT:SW_PUSH_6mm" H 1450 3500 50  0001 C CNN
 F 3 "http://www.apem.com/int/index.php?controller=attachment&id_attachment=488" H 1450 3500 50  0001 C CNN
 	1    1450 3300
