File: hardware/hardware.kicad_pcb (KiCad board)
At the start: 2 copper layers, 15 parts, among them J1 Raspberry_Pi_2_3, J2 SSD1608_SPI, J3 0906-1, J4 0906-1, J5 Batt, J6 USB_A, SW1 SW_MEC_5G, U1 MCP73871, U2 L7805

Commit message: update pcb
Parts:
- added S1: 5-Way, Sparkfun:COM-10063, F.Cu at (169.0, 111.5)
- J1: footprint Connector_PinHeader_2.54mm:PinHeader_2x20_P2.54mm_Vertical -> Connector_PinSocket_2.54mm:PinSocket_2x20_P2.54mm_Vertical
- J5, J6, U2: moved to B.Cu
- R1, R2, R3, R4, R5, R6: footprint Resistor_SMD:R_1020_2550Metric -> Resistor_SMD:R_0805_2012Metric
- SW1: footprint Button_Switch_THT:SW_Tactile_SPST_Angled_PTS645Vx31-2LFS -> Button_Switch_THT:SW_PUSH_6mm
- moved J6 171.5 mm to (179.0, 92.5), turned to 0 degrees
- moved J1 152.2 mm to (166.6, 83.2), turned to 270 degrees
- moved J3 118.5 mm to (135.0, 105.7), turned to 180 degrees
- moved J4 114.3 mm to (132.8, 105.7), turned to 180 degrees
- moved SW1 106.3 mm to (121.0, 114.5), turned to 180 degrees
- moved J5 101.1 mm to (115.0, 97.5), turned to 90 degrees
- moved U2 81.4 mm to (136.0, 112.5), turned to 180 degrees
- moved J2 68.5 mm to (134.9, 89.7)
- moved R1 65.3 mm to (158.9, 97.0), turned to 270 degrees
- moved U1 63.2 mm to (154.8, 96.8)
- moved R5 60.5 mm to (161.5, 97.1), turned to 270 degrees
- moved R4 58.4 mm to (153.4, 105.7)
- moved R2 58.4 mm to (150.0, 98.3), turned to 90 degrees
- moved R3 50.8 mm to (150.3, 94.7), turned to 90 degrees
- moved R6 48.8 mm to (153.4, 102.5)
Connections:
- SW1 pad 2: GND -> Net-(J1-Pad40)
Routing:
- net GND: track 22.2 -> 199.9 mm, vias 0 -> 4
- net Net-(J1-Pad36): track 0.00 -> 92.1 mm, vias 0 -> 2
- net Net-(J1-Pad35): track 0.00 -> 79.7 mm
- net Net-(J1-Pad38): track 0.00 -> 73.9 mm, vias 0 -> 3
- net Net-(J5-Pad2): track 0.00 -> 46.0 mm, vias 0 -> 1
- net /SPI_RESET: track 55.3 -> 10.6 mm
- net Net-(J4-Pad1): track 0.00 -> 42.5 mm
- net Net-(J3-Pad1): track 0.00 -> 40.4 mm
- net /OLED_CS: track 51.5 -> 11.7 mm
- net Net-(J1-Pad12): track 0.00 -> 38.3 mm, vias 0 -> 3
- net /SPI_DC: track 55.3 -> 17.5 mm
- net Net-(J1-Pad40): track 0.00 -> 36.9 mm
- net VBUS: track 0.00 -> 35.3 mm, vias 0 -> 5
- net Net-(J1-Pad11): track 0.00 -> 33.7 mm, vias 0 -> 3
- net /SPI_CLK: track 40.5 -> 7.02 mm
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- added copper zone on F.Cu, net GND
Other:
- board outline added: 65 x 47 mm
